Commit message: fix: seed_r7 ros2 convert

File: seed_r7_description/typef/noid.urdf.xacro (robot description, xacro)
@@ -1,4 +1,15 @@
 <?xml version="1.0"?>
 <robot name="SEED-Noid-Mover-typeF" xmlns:xacro="http://ros.org/wiki/xacro">
+  <!-- ros2_control hardware parameters (overridable from launch) -->
+  <xacro:arg name="port_upper"             default="/dev/aero_upper"/>
+  <xacro:arg name="port_lower"             default="/dev/aero_lower"/>
+  <xacro:arg name="robot_model_plugin"     default="seed_r7_robot_interface/typef"/>
+  <xacro:arg name="controller_rate"        default="50"/>
+  <xacro:arg name="overlap_scale"          default="2.0"/>
+  <xacro:arg name="joint_settings_file"    default=""/>
+  <!-- Gazebo controller params file (required when use_gazebo:=true) -->
+  <xacro:arg name="controller_params_file" default=""/>
+  <!-- Set to true to use gazebo_ros2_control hardware instead of real hardware -->
+  <xacro:arg name="use_gazebo" default="false"/>
   <!-- The following included files set up definitions of parts of the robot body -->
   <!-- wraps upperbody and hand-->
@@ -28,11 +39,151 @@
  <xacro:gazebo_laser_sensor link_name="wheels_base_laser_link"
                             frame_name="wheels_base_laser_link" />
- <!-- joint control -->
- <xacro:gazebo_trajectory_controller />
- <!-- mobile base -->
+ <!-- joint control (Gazebo only) -->
+ <xacro:gazebo_trajectory_controller controller_params_file="$(arg controller_params_file)"/>
+ <!-- mobile base (Gazebo only) -->
  <xacro:gazebo_base_controller base_frame="base_link" />
+ <!-- ========== ros2_control hardware interface ========== -->
+ <ros2_control name="seed_r7_hardware" type="system">
+   <hardware>
+     <xacro:if value="$(arg use_gazebo)">
+       <plugin>gazebo_ros2_control/GazeboSystem</plugin>
+     </xacro:if>
+     <xacro:unless value="$(arg use_gazebo)">
+       <plugin>seed_r7_ros_controller/RobotHW</plugin>
+       <param name="port_upper">$(arg port_upper)</param>
+       <param name="port_lower">$(arg port_lower)</param>
+       <param name="robot_model_plugin">$(arg robot_model_plugin)</param>
+       <param name="controller_rate">$(arg controller_rate)</param>
+       <param name="overlap_scale">$(arg overlap_scale)</param>
+       <param name="csv_config_dir">$(find seed_r7_description)/csv</param>
+       <param name="joint_settings_file">$(arg joint_settings_file)</param>
+     </xacro:unless>
+   </hardware>
+   <!-- upper body joints (22) -->
+   <joint name="waist_y_joint">
+     <command_interface name="position"/>
+     <state_interface name="position"/>
+     <state_interface name="velocity"/>
+   </joint>
+   <joint name="waist_p_joint">
+     <command_interface name="position"/>
+     <state_interface name="position"/>
+     <state_interface name="velocity"/>
+   </joint>
+   <joint name="waist_r_joint">
+     <command_interface name="position"/>
+     <state_interface name="position"/>
+     <state_interface name="velocity"/>
+   </joint>
+   <joint name="l_shoulder_p_joint">
+     <command_interface name="position"/>
+     <state_interface name="position"/>
+     <state_interface name="velocity"/>
+   </joint>
+   <joint name="l_shoulder_r_joint">
+     <command_interface name="position"/>
+     <state_interface name="position"/>
+     <state_interface name="velocity"/>
+   </joint>
+   <joint name="l_shoulder_y_joint">
+     <command_interface name="position"/>
+     <state_interface name="position"/>
+     <state_interface name="velocity"/>
+   </joint>
+   <joint name="l_elbow_joint">
+     <command_interface name="position"/>
+     <state_interface name="position"/>
+     <state_interface name="velocity"/>
+   </joint>
+   <joint name="l_wrist_y_joint">
+     <command_interface name="position"/>
+     <state_interface name="position"/>
+     <state_interface name="velocity"/>
+   </joint>
+   <joint name="l_wrist_p_joint">
+     <command_interface name="position"/>
+     <state_interface name="position"/>
+     <state_interface name="velocity"/>
+   </joint>
+   <joint name="l_wrist_r_joint">
+     <command_interface name="position"/>
+     <state_interface name="position"/>
+     <state_interface name="velocity"/>
+   </joint>
+   <joint name="l_thumb_joint">
+     <command_interface name="position"/>
+     <state_interface name="position"/>
+     <state_interface name="velocity"/>
+   </joint>
+   <joint name="neck_y_joint">
+     <command_interface name="position"/>
+     <state_interface name="position"/>
+     <state_interface name="velocity"/>
+   </joint>
+   <joint name="neck_p_joint">
+     <command_interface name="position"/>
+     <state_interface name="position"/>
+     <state_interface name="velocity"/>
+   </joint>
+   <joint name="neck_r_joint">
+     <command_interface name="position"/>
+     <state_interface name="position"/>
+     <state_interface name="velocity"/>
+   </joint>
+   <joint name="r_shoulder_p_joint">
+     <command_interface name="position"/>
+     <state_interface name="position"/>
+     <state_interface name="velocity"/>
+   </joint>
+   <joint name="r_shoulder_r_joint">
+     <command_interface name="position"/>
+     <state_interface name="position"/>
+     <state_interface name="velocity"/>
+   </joint>
+   <joint name="r_shoulder_y_joint">
+     <command_interface name="position"/>
+     <state_interface name="position"/>
+     <state_interface name="velocity"/>
+   </joint>
+   <joint name="r_elbow_joint">
+     <command_interface name="position"/>
+     <state_interface name="position"/>
+     <state_interface name="velocity"/>
+   </joint>
+   <joint name="r_wrist_y_joint">
+     <command_interface name="position"/>
+     <state_interface name="position"/>
+     <state_interface name="velocity"/>
+   </joint>
+   <joint name="r_wrist_p_joint">
+     <command_interface name="position"/>
+     <state_interface name="position"/>
+     <state_interface name="velocity"/>
+   </joint>
+   <joint name="r_wrist_r_joint">
+     <command_interface name="position"/>
+     <state_interface name="position"/>
+     <state_interface name="velocity"/>
+   </joint>
+   <joint name="r_thumb_joint">
+     <command_interface name="position"/>
+     <state_interface name="position"/>
+     <state_interface name="velocity"/>
+   </joint>
+   <!-- lower body joints (2) -->
+   <joint name="knee_joint">
+     <command_interface name="position"/>
+     <state_interface name="position"/>
+     <state_interface name="velocity"/>
+   </joint>
+   <joint name="ankle_joint">
+     <command_interface name="position"/>
+     <state_interface name="position"/>
+     <state_interface name="velocity"/>
+   </joint>
+ </ros2_control>
  <!-- mimic joints -->
  <gazebo>
-   <plugin name="mimic_updater" filename="libmimic_plugin.so">
+   <plugin filename="libmimic_plugin.so" name="mimicplugin::MimicPlugin">
      <!-- lifter -->
      <mimic joint="knee_joint"  offset="0.0" multiplier="-1.0"

File: seed_r7_description/urdf/gazebo.xacro (robot description, xacro)
@@ -31,18 +31,18 @@
     <xacro:gazebo_joint_reference joint_name="${joint_name}" />
   </xacro:macro>
-  <xacro:macro name="gazebo_trajectory_controller" params="namespace:=/" >
+  <xacro:macro name="gazebo_trajectory_controller" params="controller_params_file namespace:=/" >
     <gazebo>
-      <plugin name="gazebo_ros_control" filename="libgazebo_ros_control.so">
-        <robotNamespace>${namespace}</robotNamespace>
-        <robotSimType>gazebo_ros_control/DefaultRobotHWSim</robotSimType>
-        <legacyModeNS>true</legacyModeNS>
+      <plugin filename="gz_ros2_control" name="gz_ros2_control::GazeboSimROS2ControlPlugin">
+        <parameters>${controller_params_file}</parameters>
+        <ros>
+          <namespace>${namespace}</namespace>
+        </ros>
       </plugin>
     </gazebo>
   </xacro:macro>
   <xacro:macro name="gazebo_base_controller" params="base_frame com_topic:=/cmd_vel odom_topic:=/odom odom_frame:=odom odom_rate:=20" >
-    <!-- Base control -->
+    <!-- Base control (gz-sim8) -->
     <gazebo>
-      <!--plugin name="cmd_vel_controller" filename="libgazebo_ros_planar_force_move.so"-->
-      <plugin name="cmd_vel_controller" filename="libgazebo_ros_planar_force_move.so">
+      <plugin filename="libgazebo_ros_planar_force_move.so" name="gazebo::GazeboRosPlanarForceMove">
         <commandTopic>cmd_vel</commandTopic>
         <odometryTopic>odom</odometryTopic>

File: seed_r7_description/urdf/seed_hand/seed_hand.urdf.xacro (robot description, xacro)
@@ -53,6 +53,7 @@
     <inertial>
       <mass value="0.1" />
-      <origin xyz="0 0 -0.023" rpy="0 -0 0"/>
-      <inertia ixx="0.0001" iyy="0.0001" izz="0.0001" ixy="0" ixz="0" iyz="0" />
+      <origin xyz="0 0 -0.023" rpy="0 0 0"/>
+      <!-- box 0.020 x 0.0615 x 0.054 inertia (x10 safety margin) -->
+      <inertia ixx="0.001" iyy="0.001" izz="0.001" ixy="0" ixz="0" iyz="0" />
     </inertial>
   </link>
@@ -61,6 +62,6 @@
     <inertial>
       <mass value="0.1" />
-      <origin xyz="0 0 -0.023" rpy="0 -0 0"/>
-      <inertia ixx="0.0001" iyy="0.0001" izz="0.0001" ixy="0" ixz="0" iyz="0" />
+      <origin xyz="0 0 -0.023" rpy="0 0 0"/>
+      <inertia ixx="0.001" iyy="0.001" izz="0.001" ixy="0" ixz="0" iyz="0" />
     </inertial>
   </link>
@@ -82,6 +83,8 @@
     <inertial>
       <mass value="0.07" />
-      <origin xyz="0 ${reflect * 0.014} -0.0225" rpy="0 -0 0"/>
-      <inertia ixx="0.0014" iyy="0.0001" izz="0.0001" ixy="0" ixz="0" iyz="0" />
+      <origin xyz="0 ${reflect * 0.014} -0.0225" rpy="0 0 0"/>
+      <!-- Fixed: was ixx=0.0014 which violated triangle inequality (ixx > iyy+izz) -->
+      <!-- box 0.020 x 0.0596 x 0.065 inertia (x10 safety margin) -->
+      <inertia ixx="0.001" iyy="0.001" izz="0.001" ixy="0" ixz="0" iyz="0" />
     </inertial>
   </link>
@@ -103,6 +106,7 @@
     <inertial>
       <mass value="0.1" />
-      <origin xyz="0 0 -0.04" rpy="0 -0 0"/>
-      <inertia ixx="0.0001" iyy="0.0001" izz="0.0001" ixy="0" ixz="0" iyz="0" />
+      <origin xyz="0 0 -0.04" rpy="0 0 0"/>
+      <!-- box 0.032 x 0.054 x 0.105 inertia (x10 safety margin) -->
+      <inertia ixx="0.001" iyy="0.001" izz="0.001" ixy="0" ixz="0" iyz="0" />
     </inertial>
   </link>
